Commit message: cambios: - corregido el modelo - ahora el modelo puede hacer reversa - añadida configuración de rviz - añadido nodo para teleoperacion

File: urdf/modelo.urdf (robot description, URDF)
Before this commit: robot quad_ackermann_viewer_safe, 12 links, 11 joints
Links:
- link base_link: geometry collision box size=0.80 0.45 0.12; visual box size=0.80 0.45 0.12
- link camera_link: mass None -> 0.1; geometry collision box size=0.06 0.04 0.04; visual box size=0.06 0.04 0.04
- link front_left_steer_link: mass None -> 0.5; geometry collision box size=0.06 0.04 0.10; visual box size=0.06 0.04 0.10
- link front_left_wheel_link: mass None -> 1.0
- link front_right_steer_link: mass None -> 0.5; geometry collision box size=0.06 0.04 0.10; visual box size=0.06 0.04 0.10
- link front_right_wheel_link: mass None -> 1.0
- link gps_link: mass None -> 0.05
- link imu_link: mass None -> 0.05
- link lidar_link: mass None -> 0.1; geometry collision cylinder length=0.06 radius=0.05; visual cylinder length=0.06 radius=0.05
- link rear_left_wheel_link: mass None -> 1.0
- link rear_right_wheel_link: mass None -> 1.0
Joints:
- joint camera_joint: origin xyz=0.40 0.0 0.40 rpy=0 0 0 -> xyz=0.40 0.0 0.32 rpy=0 0 0
- joint front_left_steer_joint: origin xyz=0.30 0.24 0.15 rpy=0 0 0 -> xyz=0.30 0.28 0.15 rpy=0 0 0
- joint front_right_steer_joint: origin xyz=0.30 -0.24 0.15 rpy=0 0 0 -> xyz=0.30 -0.28 0.15 rpy=0 0 0
- joint gps_joint: origin xyz=0.0 0.0 0.45 rpy=0 0 0 -> xyz=0.0 0.0 0.34 rpy=0 0 0
- joint imu_joint: origin xyz=0.0 0.0 0.35 rpy=0 0 0 -> xyz=0.0 0.0 0.30 rpy=0 0 0
- joint lidar_joint: origin xyz=0.20 0.0 0.45 rpy=0 0 0 -> xyz=0.20 0.0 0.33 rpy=0 0 0
- joint rear_left_wheel_joint: origin xyz=-0.30 0.24 0.15 rpy=0 0 0 -> xyz=-0.30 0.28 0.15 rpy=0 0 0
- joint rear_right_wheel_joint: origin xyz=-0.30 -0.24 0.15 rpy=0 0 0 -> xyz=-0.30 -0.28 0.15 rpy=0 0 0

Commit message: mejoras en los parametros de navegación; sigue sin poder navegar autonomamente

File: urdf/modelo.urdf (robot description, URDF)
Before this commit: robot quad_ackermann_viewer_safe, 12 links, 11 joints
Joints:
- joint front_left_steer_joint: limit lower=-0.5235987756 upper=0.5235987756 effort=50 velocity=2.0 -> lower=-0.5235987756 upper=0.5235987756 effort=50 velocity=5.0
- joint front_right_steer_joint: limit lower=-0.5235987756 upper=0.5235987756 effort=50 velocity=2.0 -> lower=-0.5235987756 upper=0.5235987756 effort=50 velocity=5.0
