Commit message: cambios en parametros

File: urdf/cuatri.urdf (robot description, URDF)
Before this commit: robot quad_ackermann_viewer_safe, 12 links, 11 joints
Links:
- link base_link: mass 20.0 -> 50.0; geometry collision box size=1.20 0.60 0.25; visual box size=1.20 0.60 0.25
- link front_left_steer_link: geometry collision box size=0.10 0.08 0.15; visual box size=0.10 0.08 0.15
- link front_left_wheel_link: mass 1.0 -> 2.0; geometry collision cylinder length=0.16 radius=0.24; visual cylinder length=0.16 radius=0.24
- link front_right_steer_link: geometry collision box size=0.10 0.08 0.15; visual box size=0.10 0.08 0.15
- link front_right_wheel_link: mass 1.0 -> 2.0; geometry collision cylinder length=0.16 radius=0.24; visual cylinder length=0.16 radius=0.24
- link rear_left_wheel_link: mass 1.0 -> 2.0; geometry collision cylinder length=0.16 radius=0.24; visual cylinder length=0.16 radius=0.24
- link rear_right_wheel_link: mass 1.0 -> 2.0; geometry collision cylinder length=0.16 radius=0.24; visual cylinder length=0.16 radius=0.24
Joints:
- joint camera_joint: origin xyz=0.40 0.0 0.32 rpy=0 0 0 -> xyz=0.50 0.0 0.60 rpy=0 0 0
- joint front_left_steer_joint: limit lower=-0.5235987756 upper=0.5235987756 effort=50 velocity=5.0 -> lower=-0.5235987756 upper=0.5235987756 effort=100 velocity=2.0; origin xyz=0.30 0.28 0.15 rpy=0 0 0 -> xyz=0.47 0.375 0.24 rpy=0 0 0
- joint front_left_wheel_joint: limit lower=-1000 upper=1000 effort=100 velocity=100 -> lower=-1000 upper=1000 effort=200 velocity=100
- joint front_right_steer_joint: limit lower=-0.5235987756 upper=0.5235987756 effort=50 velocity=5.0 -> lower=-0.5235987756 upper=0.5235987756 effort=100 velocity=2.0; origin xyz=0.30 -0.28 0.15 rpy=0 0 0 -> xyz=0.47 -0.375 0.24 rpy=0 0 0
- joint front_right_wheel_joint: limit lower=-1000 upper=1000 effort=100 velocity=100 -> lower=-1000 upper=1000 effort=200 velocity=100
- joint gps_joint: origin xyz=0.0 0.0 0.34 rpy=0 0 0 -> xyz=0.0 0.0 0.62 rpy=0 0 0
- joint imu_joint: origin xyz=0.0 0.0 0.30 rpy=0 0 0 -> xyz=0.0 0.0 0.58 rpy=0 0 0
- joint lidar_joint: origin xyz=0.20 0.0 0.45 rpy=0 0 0 -> xyz=0.30 0.0 0.65 rpy=0 0 0
- joint rear_left_wheel_joint: limit lower=-1000 upper=1000 effort=100 velocity=100 -> lower=-1000 upper=1000 effort=200 velocity=100; origin xyz=-0.30 0.28 0.15 rpy=0 0 0 -> xyz=-0.47 0.375 0.24 rpy=0 0 0
- joint rear_right_wheel_joint: limit lower=-1000 upper=1000 effort=100 velocity=100 -> lower=-1000 upper=1000 effort=200 velocity=100; origin xyz=-0.30 -0.28 0.15 rpy=0 0 0 -> xyz=-0.47 -0.375 0.24 rpy=0 0 0

Commit message: mejoras en la configuración de nav2

File: urdf/cuatri.urdf (robot description, URDF)
Before this commit: robot quad_ackermann_viewer_safe, 12 links, 11 joints
Joints:
- joint camera_joint: origin xyz=0.50 0.0 0.60 rpy=0 0 0 -> xyz=0.97 0.0 0.60 rpy=0 0 0
- joint front_left_steer_joint: origin xyz=0.47 0.375 0.24 rpy=0 0 0 -> xyz=0.94 0.375 0.24 rpy=0 0 0
- joint front_right_steer_joint: origin xyz=0.47 -0.375 0.24 rpy=0 0 0 -> xyz=0.94 -0.375 0.24 rpy=0 0 0
- joint gps_joint: origin xyz=0.0 0.0 0.62 rpy=0 0 0 -> xyz=0.47 0.0 0.62 rpy=0 0 0
- joint imu_joint: origin xyz=0.0 0.0 0.58 rpy=0 0 0 -> xyz=0.47 0.0 0.58 rpy=0 0 0
- joint lidar_joint: origin xyz=0.30 0.0 0.65 rpy=0 0 0 -> xyz=0.77 0.0 0.65 rpy=0 0 0
- joint rear_left_wheel_joint: origin xyz=-0.47 0.375 0.24 rpy=0 0 0 -> xyz=0.0 0.375 0.24 rpy=0 0 0
- joint rear_right_wheel_joint: origin xyz=-0.47 -0.375 0.24 rpy=0 0 0 -> xyz=0.0 -0.375 0.24 rpy=0 0 0

Commit message: cambios: - eliminada la camara - ajustes en parametros

File: urdf/cuatri.urdf (robot description, URDF)
Before this commit: robot quad_ackermann_viewer_safe, 12 links, 11 joints
Links:
- removed link camera_link
Joints:
- removed joint camera_joint
