Commit message: cambios: - añadido el modelo con ultrasonidos (no funciona) - cambios en parametros

File: models/cuatri_ultrasound.urdf (robot description, URDF)
Before this commit: robot quad_ackermann_viewer_safe, 11 links, 10 joints
Links:
- added link front_left_ultrasound, mass 0.02; collision cylinder length=0.01 radius=0.04; visual cylinder length=0.01 radius=0.04
- added link front_right_ultrasound, mass 0.02; collision cylinder length=0.01 radius=0.04; visual cylinder length=0.01 radius=0.04
- added link rear_center_ultrasound, mass 0.02; collision cylinder length=0.01 radius=0.04; visual cylinder length=0.01 radius=0.04
- added link rear_left_ultrasound, mass 0.02; collision cylinder length=0.01 radius=0.04; visual cylinder length=0.01 radius=0.04
- added link rear_right_ultrasound, mass 0.02; collision cylinder length=0.01 radius=0.04; visual cylinder length=0.01 radius=0.04
Joints:
- added joint front_left_ultrasound_joint: type fixed, parent base_link, child front_left_ultrasound, origin xyz=1.05 0.25 0.35 rpy=0 0 0
- added joint front_right_ultrasound_joint: type fixed, parent base_link, child front_right_ultrasound, origin xyz=1.05 -0.25 0.35 rpy=0 0 0
- added joint rear_center_ultrasound_joint: type fixed, parent base_link, child rear_center_ultrasound, origin xyz=-0.10 0.0 0.35 rpy=0 0 3.14159265359
- added joint rear_left_ultrasound_joint: type fixed, parent base_link, child rear_left_ultrasound, origin xyz=-0.10 0.25 0.35 rpy=0 0 3.14159265359
- added joint rear_right_ultrasound_joint: type fixed, parent base_link, child rear_right_ultrasound, origin xyz=-0.10 -0.25 0.35 rpy=0 0 3.14159265359
