Commit message: cambios en parametros

File: models/cuatri_real.urdf (robot description, URDF)
Before this commit: robot quad_ackermann_viewer_safe, 11 links, 10 joints
Joints:
- joint front_left_steer_joint: limit lower=-0.5235987756 upper=0.5235987756 effort=100 velocity=2.0 -> lower=-0.5235987756 upper=0.5235987756 effort=100 velocity=5.0
- joint front_right_steer_joint: limit lower=-0.5235987756 upper=0.5235987756 effort=100 velocity=2.0 -> lower=-0.5235987756 upper=0.5235987756 effort=100 velocity=5.0

Commit message: parametros v2

File: models/cuatri_real.urdf (robot description, URDF)
Before this commit: robot quad_ackermann_viewer_safe, 11 links, 10 joints
Joints:
- joint front_left_steer_joint: limit lower=-0.5235987756 upper=0.5235987756 effort=100 velocity=5.0 -> lower=-0.5235987756 upper=0.5235987756 effort=100 velocity=3.0
- joint front_right_steer_joint: limit lower=-0.5235987756 upper=0.5235987756 effort=100 velocity=5.0 -> lower=-0.5235987756 upper=0.5235987756 effort=100 velocity=3.0

Commit message: añadida friccion mas realista a la simulacion y unos rayos blancos a las ruedas del modelo

File: models/cuatri_real.urdf (robot description, URDF)
Before this commit: robot quad_ackermann_viewer_safe, 11 links, 10 joints
Links:
- link front_left_wheel_link: geometry collision cylinder length=0.16 radius=0.24; visual box size=0.24 0.018 0.018
- link front_right_wheel_link: geometry collision cylinder length=0.16 radius=0.24; visual box size=0.24 0.018 0.018
- link rear_left_wheel_link: geometry collision cylinder length=0.16 radius=0.24; visual box size=0.24 0.018 0.018
- link rear_right_wheel_link: geometry collision cylinder length=0.16 radius=0.24; visual box size=0.24 0.018 0.018

Commit message: Unify single and dual GPS navigation flow

File: models/cuatri_real.urdf (robot description, URDF)
Before this commit: robot quad_ackermann_viewer_safe, 11 links, 10 joints
Links:
- added link gps1_link, mass 0.05; visual box size=0.07 0.04 0.035
- added link gps2_link, mass 0.05; visual box size=0.07 0.04 0.035
Joints:
- added joint gps1_joint: type fixed, parent base_link, child gps1_link, origin xyz=0.94 0.0 0.65 rpy=0 0 0
- added joint gps2_joint: type fixed, parent base_link, child gps2_link, origin xyz=0.0 0.0 0.65 rpy=0 0 0
